Commit message: temp

File: resources/robots/go2w_description/urdf/go2w_description.urdf (robot description, URDF)
Before this commit: robot go2w_description, 33 links, 32 joints
Joints:
- joint FL_foot_joint: type continuous -> revolute
- joint FR_foot_joint: type continuous -> revolute
- joint RL_foot_joint: type continuous -> revolute
- joint RR_foot_joint: type continuous -> revolute

File: resources/robots/go2w_piper_description/urdf/go2w_piper_description.urdf (robot description, URDF)
Before this commit: robot go2w_piper_description, 43 links, 42 joints
Joints:
- joint FL_foot_joint: type continuous -> revolute
- joint FR_foot_joint: type continuous -> revolute
- joint RL_foot_joint: type continuous -> revolute
- joint RR_foot_joint: type continuous -> revolute

Commit message: wheel collision model is modified to the cylinder

File: resources/robots/go2w_description/urdf/go2w_description.urdf (robot description, URDF)
Before this commit: robot go2w_description, 33 links, 32 joints
Links:
- link FL_foot: geometry collision cylinder length=0.048 radius=0.086; visual mesh filename=../dae/left_wheel.dae
- link FR_foot: geometry collision cylinder length=0.048 radius=0.086; visual mesh filename=../dae/right_wheel.dae
- link RL_foot: geometry collision cylinder length=0.048 radius=0.086; visual mesh filename=../dae/left_wheel.dae
- link RR_foot: geometry collision cylinder length=0.048 radius=0.086; visual mesh filename=../dae/right_wheel.dae

File: resources/robots/go2w_piper_description/urdf/go2w_piper_description.urdf (robot description, URDF)
Before this commit: robot go2w_piper_description, 43 links, 42 joints
Links:
- link FL_foot: geometry collision cylinder length=0.048 radius=0.086; visual mesh filename=../meshes/go2w/left_wheel.dae
- link FR_foot: geometry collision cylinder length=0.048 radius=0.086; visual mesh filename=../meshes/go2w/right_wheel.dae
- link RL_foot: geometry collision cylinder length=0.048 radius=0.086; visual mesh filename=../meshes/go2w/left_wheel.dae
- link RR_foot: geometry collision cylinder length=0.048 radius=0.086; visual mesh filename=../meshes/go2w/right_wheel.dae
