Commit message: add env_test

File: resources/robots/go2w_piper_description/urdf/go2w_piper_description.urdf (robot description, URDF)
Before this commit: robot go2w_piper_description, 43 links, 42 joints
Joints:
- joint joint7: type prismatic -> fixed
- joint joint8: type prismatic -> fixed

Commit message: add arm control

File: resources/robots/go2w_piper_description/urdf/go2w_piper_description.urdf (robot description, URDF)
Before this commit: robot go2w_piper_description, 43 links, 42 joints
Links:
- link link4: geometry visual mesh filename=../meshes/piper/dae/link4.dae

Commit message: changed piper urdf

File: resources/robots/go2w_piper_description/urdf/go2w_piper_description.urdf (robot description, URDF)
Before this commit: robot go2w_piper_description, 43 links, 42 joints
Links:
- removed link Head_lower
- removed link Head_upper
- removed link hand_cam
- removed link imu
- removed link radar
- added link gripper_base, mass 0.45; collision mesh filename=../meshes/piper/gripper_base.STL; visual mesh filename=../meshes/piper/gripper_base.STL
- link arm_base: mass 10.162548567403693 -> 1.02; geometry collision mesh filename=../meshes/piper/base_link.STL; visual mesh filename=../meshes/piper/base_link.STL
- link link1: mass 0.0978679932242825 -> 0.71; geometry collision mesh filename=../meshes/piper/link1.STL; visual mesh filename=../meshes/piper/link1.STL
- link link2: mass 0.290888938633388 -> 1.17; geometry collision mesh filename=../meshes/piper/link2.STL; visual mesh filename=../meshes/piper/link2.STL
- link link3: mass 0.290847697793211 -> 0.5; geometry collision mesh filename=../meshes/piper/link3.STL; visual mesh filename=../meshes/piper/link3.STL
- link link4: mass 0.127087348341362 -> 0.38; geometry collision mesh filename=../meshes/piper/link4.STL; visual mesh filename=../meshes/piper/link4.STL
- link link5: mass 0.144711242639457 -> 0.383; geometry collision mesh filename=../meshes/piper/link5.STL; visual mesh filename=../meshes/piper/link5.STL
- link link6: mass 0.195187143240719 -> 0.007; geometry collision mesh filename=../meshes/piper/link6.STL; visual mesh filename=../meshes/piper/link6.STL
- link link7: mass 0.02648229234527 -> 0.025; geometry collision mesh filename=../meshes/piper/link7.STL; visual mesh filename=../meshes/piper/link7.STL
- link link8: mass 0.0264822021416248 -> 0.025; geometry collision mesh filename=../meshes/piper/link8.STL; visual mesh filename=../meshes/piper/link8.STL
Joints:
- removed joint Head_lower_joint
- removed joint Head_upper_joint
- removed joint hand_camera_joint
- removed joint imu_joint
- removed joint radar_joint
- added joint joint6_to_gripper_base: type fixed, parent link6, child gripper_base, origin xyz=0 0 0 rpy=0 0 0
- joint base2arm: origin xyz=0 0 0.06 rpy=0 0 0 -> xyz=0 0 0.05 rpy=0 0 0
- joint joint1: limit lower=-2.618 upper=2.618 effort=100 velocity=3 -> lower=-2.618 upper=2.618 effort=100 velocity=5; origin xyz=0 0 0.123 rpy=0 0 -1.5708 -> xyz=0 0 0.123 rpy=0 0 0
- joint joint2: limit lower=0 upper=3.14 effort=100 velocity=3 -> lower=0 upper=3.14 effort=100 velocity=5; origin xyz=0 0 0 rpy=1.5708 -0.034907 -1.5708 -> xyz=0 0 0 rpy=1.5708 -0.1359 -3.1416
- joint joint3: limit lower=-2.697 upper=0 effort=100 velocity=3 -> lower=-2.967 upper=0 effort=100 velocity=5; origin xyz=0.28358 0.028726 0 rpy=0 0 0.06604341 -> xyz=0.28503 0 0 rpy=0 0 -1.7939
- joint joint4: limit lower=-1.832 upper=1.832 effort=100 velocity=3 -> lower=-1.745 upper=1.745 effort=100 velocity=5; origin xyz=-0.24221 0.068514 0 rpy=-1.5708 0 1.3826 -> xyz=-0.021984 -0.25075 0 rpy=1.5708 0 0
- joint joint5: limit lower=-1.22 upper=1.22 effort=100 velocity=3 -> lower=-1.22 upper=1.22 effort=100 velocity=5; origin xyz=0 0 0 rpy=1.5708 0 0 -> xyz=0 0 0 rpy=-1.5708 0 0
- joint joint6: limit lower=-3.14 upper=3.14 effort=100 velocity=3 -> lower=-2.0944 upper=2.0944 effort=100 velocity=3; origin xyz=0 0.091 0.0014165 rpy=-1.5708 -1.5708 0 -> xyz=8.8259E-05 -0.091 0 rpy=1.5708 0 0
- joint joint7: axis 0 0 -1 -> 0 0 1; limit lower=0 upper=0.05 effort=100 velocity=1 -> lower=0 upper=0.035 effort=10 velocity=1; origin xyz=0 0 0.13503 rpy=1.5708 0 1.5708 -> xyz=0 0 0.1358 rpy=1.5708 0 0; parent link6 -> gripper_base
- joint joint8: axis 0 0 1 -> 0 0 -1; limit lower=-0.05 upper=0 effort=100 velocity=1 -> lower=-0.035 upper=0 effort=10 velocity=1; origin xyz=0 0 0.13503 rpy=-1.5708 0 1.5708 -> xyz=0 0 0.1358 rpy=1.5708 0 -3.1416; parent link6 -> gripper_base

Commit message: change reward weights

File: resources/robots/go2w_piper_description/urdf/go2w_piper_description.urdf (robot description, URDF)
Before this commit: robot go2w_piper_description, 39 links, 38 joints
Joints:
- joint base2arm: origin xyz=0 0 0.05 rpy=0 0 0 -> xyz=0.1 0 0.05 rpy=0 0 0
